Commit message: ur5e4

File: src/my_arm_description/urdf/my_arm_ur5e2.urdf.xacro (robot description, xacro)
@@ -14,6 +14,6 @@
   -->
   <xacro:arg name="d1" default="0.1625"/>
-  <xacro:arg name="a2" default="0.425"/>
-  <xacro:arg name="a3" default="0.3922"/>
+  <xacro:arg name="a2" default="-0.425"/>
+  <xacro:arg name="a3" default="-0.3922"/>
   <xacro:arg name="d4" default="0.1333"/>
   <xacro:arg name="d5" default="0.0997"/>
@@ -33,6 +33,6 @@
   <!-- Convenience properties -->
   <xacro:property name="d1" value="$(arg d1)"/>
-  <xacro:property name="a2" value="$(arg a2)"/>
-  <xacro:property name="a3" value="$(arg a3)"/>
+  <xacro:property name="a2_len" value="${-1.0 * $(arg a2)}"/>
+  <xacro:property name="a3_len" value="${-1.0 * $(arg a3)}"/>
   <xacro:property name="d4" value="$(arg d4)"/>
   <xacro:property name="d5" value="$(arg d5)"/>
@@ -127,6 +127,6 @@
   <!-- Physical links (simple geometry) -->
   <xacro:cyl_z name="link1" length="${d1}" mat="grey" mass="$(arg m_link)"/>
-  <xacro:cyl_x name="link2" length="${a2}" mat="grey" mass="$(arg m_link)"/>
-  <xacro:cyl_x name="link3" length="${a3}" mat="grey" mass="$(arg m_link)"/>
+  <xacro:cyl_x name="link2" length="${a2_len}" mat="grey" mass="$(arg m_link)"/>
+  <xacro:cyl_x name="link3" length="${a3_len}" mat="grey" mass="$(arg m_link)"/>
   <xacro:cyl_z name="link4" length="${d4}" mat="blue" mass="$(arg m_link)"/>
   <xacro:cyl_z name="link5" length="${d5}" mat="blue" mass="$(arg m_link)"/>
@@ -163,5 +163,11 @@
     <parent link="frame1"/>
     <child link="link1"/>
-    <origin xyz="0 0 ${d1}" rpy="1.57079632679 0 0"/>
+    <origin xyz="0 0 ${d1}" rpy="0 0 0"/>
+  </joint>
+  <link name="frame1_twist"/>
+  <joint name="dh1_twist" type="fixed">
+    <parent link="link1"/>
+    <child link="frame1_twist"/>
+    <origin xyz="0 0 0" rpy="1.57079632679 0 0"/>
   </joint>
   <!-- Joint 2: rotation about Z (DH theta2) -->

Commit message: ur5e6

File: src/my_arm_description/urdf/my_arm_ur5e2.urdf.xacro (robot description, xacro)
@@ -1,43 +1,29 @@
 <?xml version="1.0"?>
-<robot xmlns:xacro="http://ros.org/wiki/xacro" name="ur5e_simple_dh">
+<robot xmlns:xacro="http://ros.org/wiki/xacro" name="ur5e_simple">
   <xacro:arg name="ros2_control_params" default=""/>
-  <!--
-       UR5e DH parameters (meters)
-       (Common UR5e table; a2,a3 are negative in DH. Here we keep their magnitudes
-        and apply the sign in the fixed transforms.)
-       d1=0.1625
-       a2=-0.425
-       a3=-0.3922
-       d4=0.1333
-       d5=0.0997
-       d6=0.0996
-  -->
+  <!-- UR5e approximate dimensions (m) -->
   <xacro:arg name="d1" default="0.1625"/>
-  <xacro:arg name="a2" default="-0.425"/>
-  <xacro:arg name="a3" default="-0.3922"/>
+  <xacro:arg name="a2" default="0.425"/>
+  <xacro:arg name="a3" default="0.3922"/>
   <xacro:arg name="d4" default="0.1333"/>
   <xacro:arg name="d5" default="0.0997"/>
   <xacro:arg name="d6" default="0.0996"/>
-  <!-- Visual thickness / base -->
+  <!-- Visual thickness -->
   <xacro:arg name="r_link" default="0.03"/>
+  <!-- Base box -->
   <xacro:arg name="base_x" default="0.18"/>
   <xacro:arg name="base_y" default="0.18"/>
   <xacro:arg name="base_z" default="0.06"/>
-  <!-- Masses (non-zero) -->
+  <!-- Masses -->
   <xacro:arg name="m_base" default="5.0"/>
-  <xacro:arg name="m_link" default="2.0"/>
+  <xacro:arg name="m_link" default="0.8"/>   <!-- IMPORTANT: start light -->
   <xacro:arg name="m_tool" default="0.2"/>
-  <!-- Joint limits -->
+  <!-- Limits -->
   <xacro:arg name="joint_vel" default="2.0"/>
   <xacro:arg name="joint_effort" default="50.0"/>
-  <!-- Convenience properties -->
-  <xacro:property name="d1" value="$(arg d1)"/>
-  <xacro:property name="a2_len" value="${-1.0 * $(arg a2)}"/>
-  <xacro:property name="a3_len" value="${-1.0 * $(arg a3)}"/>
-  <xacro:property name="d4" value="$(arg d4)"/>
-  <xacro:property name="d5" value="$(arg d5)"/>
-  <xacro:property name="d6" value="$(arg d6)"/>
-  <xacro:property name="r"  value="$(arg r_link)"/>
-  <!--   Inertial macros (safe)    -->
+  <xacro:property name="r" value="$(arg r_link)"/>
+  <!--
+       Inertia macros
+        -->
   <xacro:macro name="inertial_box" params="mass x y z">
     <inertial>
@@ -56,5 +42,4 @@
     </inertial>
   </xacro:macro>
-  <!-- Cylinder aligned with X (visual only); inertia approx swapped -->
   <xacro:macro name="inertial_cylinder_x" params="mass radius length">
     <inertial>
@@ -65,9 +50,20 @@
     </inertial>
   </xacro:macro>
-  <!--  Materials  -->
+  <xacro:macro name="inertial_cylinder_y" params="mass radius length">
+    <inertial>
+      <mass value="${mass}"/>
+      <inertia ixx="${mass*(3*radius*radius + length*length)/12.0}" ixy="0.0" ixz="0.0"
+               iyy="${mass*(radius*radius)/2.0}" iyz="0.0"
+               izz="${mass*(3*radius*radius + length*length)/12.0}"/>
+    </inertial>
+  </xacro:macro>
+  <!--
+       Materials
+        -->
   <material name="dark"><color rgba="0.2 0.2 0.2 1.0"/></material>
-  <material name="grey"><color rgba="0.6 0.6 0.6 1.0"/></material>
-  <material name="blue"><color rgba="0.2 0.3 0.8 1.0"/></material>
-  <!--  Links   -->
+  <material name="pale_blue"><color rgba="0.6 0.75 0.95 1.0"/></material>
+  <!--
+       World + base
+        -->
   <link name="world"/>
   <joint name="world_to_base" type="fixed">
@@ -88,11 +84,13 @@
     <xacro:inertial_box mass="$(arg m_base)" x="$(arg base_x)" y="$(arg base_y)" z="$(arg base_z)"/>
   </link>
-  <!-- Helper macro: a simple cylinder "physical" link along Z -->
-  <xacro:macro name="cyl_z" params="name length mat mass">
+  <!--
+       Link macros (cylinders along x/y/z)
+        -->
+  <xacro:macro name="cyl_z" params="name length mass">
     <link name="${name}">
       <visual>
         <origin xyz="0 0 ${length/2.0}" rpy="0 0 0"/>
         <geometry><cylinder radius="${r}" length="${length}"/></geometry>
-        <material name="${mat}"/>
+        <material name="pale_blue"/>
       </visual>
       <collision>
@@ -103,14 +101,14 @@
     </link>
   </xacro:macro>
-  <!-- Helper macro: a simple cylinder "physical" link along X -->
-  <xacro:macro name="cyl_x" params="name length mat mass">
+  <xacro:macro name="cyl_x" params="name length mass sign">
+    <!-- sign: +1 or -1 to draw toward +X or -X -->
     <link name="${name}">
       <visual>
-        <origin xyz="${length/2.0} 0 0" rpy="0 1.57079632679 0"/>
-        <geometry><cylinder radius="${r}" length="${length}"/></geometry>
-        <material name="${mat}"/>
+        <origin xyz="${sign*length/2.0} 0 0" rpy="0 1.57079632679 0"/>
+        <geometry><cylinder radius="${r}" length="${length}"/></geometry>
+        <material name="pale_blue"/>
       </visual>
       <collision>
-        <origin xyz="${length/2.0} 0 0" rpy="0 1.57079632679 0"/>
+        <origin xyz="${sign*length/2.0} 0 0" rpy="0 1.57079632679 0"/>
         <geometry><cylinder radius="${r}" length="${length}"/></geometry>
       </collision>
@@ -118,139 +116,88 @@
     </link>
   </xacro:macro>
-  <!-- Frame-only links (tiny, but with inertial to avoid parser issues if you ever add collision) -->
-  <link name="frame1"/>
-  <link name="frame2"/>
-  <link name="frame3"/>
-  <link name="frame4"/>
-  <link name="frame5"/>
-  <link name="frame6"/>
-  <!-- Physical links (simple geometry) -->
-  <xacro:cyl_z name="link1" length="${d1}" mat="grey" mass="$(arg m_link)"/>
-  <xacro:cyl_x name="link2" length="${a2_len}" mat="grey" mass="$(arg m_link)"/>
-  <xacro:cyl_x name="link3" length="${a3_len}" mat="grey" mass="$(arg m_link)"/>
-  <xacro:cyl_z name="link4" length="${d4}" mat="blue" mass="$(arg m_link)"/>
-  <xacro:cyl_z name="link5" length="${d5}" mat="blue" mass="$(arg m_link)"/>
-  <xacro:cyl_z name="link6" length="${d6}" mat="blue" mass="$(arg m_link)"/>
-  <!-- Optional tool marker (fixed). Keep it if useful for TF. -->
-  <link name="tool0">
-    <visual>
-      <origin xyz="0 0 0.02" rpy="0 0 0"/>
-      <geometry><box size="0.05 0.05 0.04"/></geometry>
-      <material name="dark"/>
-    </visual>
-    <collision>
-      <origin xyz="0 0 0.02" rpy="0 0 0"/>
-      <geometry><box size="0.05 0.05 0.04"/></geometry>
-    </collision>
-    <xacro:inertial_box mass="$(arg m_tool)" x="0.05" y="0.05" z="0.04"/>
-  </link>
-  <!--
-       Joints (DH-correct structure)
-       Revolute joints are the 6 DOF joints: joint1..joint6
-       Fixed joints implement DH offsets/twists between joint frames.
-        -->
-  <!-- Joint 1: rotation about Z at base -->
+  <xacro:macro name="cyl_y" params="name length mass sign">
+    <!-- sign: +1 or -1 to draw toward +Y or -Y -->
+    <link name="${name}">
+      <visual>
+        <origin xyz="0 ${sign*length/2.0} 0" rpy="1.57079632679 0 0"/>
+        <geometry><cylinder radius="${r}" length="${length}"/></geometry>
+        <material name="pale_blue"/>
+      </visual>
+      <collision>
+        <origin xyz="0 ${sign*length/2.0} 0" rpy="1.57079632679 0 0"/>
+        <geometry><cylinder radius="${r}" length="${length}"/></geometry>
+      </collision>
+      <xacro:inertial_cylinder_y mass="${mass}" radius="${r}" length="${length}"/>
+    </link>
+  </xacro:macro>
+  <!-- Physical links -->
+  <xacro:cyl_z name="link1" length="$(arg d1)" mass="$(arg m_link)"/>
+  <xacro:cyl_x name="link2" length="$(arg a2)" mass="$(arg m_link)" sign="-1"/>
+  <xacro:cyl_x name="link3" length="$(arg a3)" mass="$(arg m_link)" sign="-1"/>
+  <!-- Wrist links oriented as you requested:
+       link4 -> -Y, link5 -> -Z, link6 -> -Y -->
+  <xacro:cyl_y name="link4" length="$(arg d4)" mass="$(arg m_link)" sign="-1"/>
+  <xacro:cyl_z name="link5" length="$(arg d5)" mass="$(arg m_link)"/>
+  <xacro:cyl_y name="link6" length="$(arg d6)" mass="$(arg m_link)" sign="-1"/>
+  <!--
+       Joints (simple, practical)
+        -->
+  <!-- joint1: base yaw -->
   <joint name="joint1" type="revolute">
     <parent link="base_link"/>
-    <child link="frame1"/>
+    <child link="link1"/>
     <origin xyz="0 0 $(arg base_z)" rpy="0 0 0"/>
     <axis xyz="0 0 1"/>
     <limit lower="-6.28318530718" upper="6.28318530718" effort="$(arg joint_effort)" velocity="$(arg joint_vel)"/>
-    <dynamics damping="0.2" friction="0.0"/>
-  </joint>
-  <!-- DH after joint1: TransZ(d1) * RotX(+pi/2) -->
-  <joint name="dh1_fixed" type="fixed">
-    <parent link="frame1"/>
-    <child link="link1"/>
-    <origin xyz="0 0 ${d1}" rpy="0 0 0"/>
-  </joint>
-  <link name="frame1_twist"/>
-  <joint name="dh1_twist" type="fixed">
-    <parent link="link1"/>
-    <child link="frame1_twist"/>
-    <origin xyz="0 0 0" rpy="1.57079632679 0 0"/>
-  </joint>
-  <!-- Joint 2: rotation about Z (DH theta2) -->
+    <dynamics damping="1.0" friction="0.0"/>
+  </joint>
+  <!-- joint2: shoulder pitch (about Y) at top of link1 -->
   <joint name="joint2" type="revolute">
     <parent link="link1"/>
-    <child link="frame2"/>
-    <origin xyz="0 0 0" rpy="0 0 0"/>
-    <axis xyz="0 0 1"/>
-    <limit lower="-6.28318530718" upper="6.28318530718" effort="$(arg joint_effort)" velocity="$(arg joint_vel)"/>
-    <dynamics damping="0.2" friction="0.0"/>
-  </joint>
-  <!-- DH after joint2: TransX(a2) (a2 is negative) -->
-  <joint name="dh2_fixed" type="fixed">
-    <parent link="frame2"/>
     <child link="link2"/>
-    <origin xyz="${a2} 0 0" rpy="0 0 0"/>
-  </joint>
-  <!-- Joint 3: rotation about Z (DH theta3) -->
+    <origin xyz="0 0 $(arg d1)" rpy="0 0 0"/>
+    <axis xyz="0 1 0"/>
+    <limit lower="-6.28318530718" upper="6.28318530718" effort="$(arg joint_effort)" velocity="$(arg joint_vel)"/>
+    <dynamics damping="2.0" friction="0.0"/>
+  </joint>
+  <!-- joint3: elbow pitch (about Y) at end of link2 (toward -X) -->
   <joint name="joint3" type="revolute">
     <parent link="link2"/>
-    <child link="frame3"/>
-    <origin xyz="0 0 0" rpy="0 0 0"/>
-    <axis xyz="0 0 1"/>
-    <limit lower="-6.28318530718" upper="6.28318530718" effort="$(arg joint_effort)" velocity="$(arg joint_vel)"/>
-    <dynamics damping="0.2" friction="0.0"/>
-  </joint>
-  <!-- DH after joint3: TransX(a3) (a3 is negative) -->
-  <joint name="dh3_fixed" type="fixed">
-    <parent link="frame3"/>
     <child link="link3"/>
-    <origin xyz="${a3} 0 0" rpy="0 0 0"/>
-  </joint>
-  <!-- Joint 4: rotation about Z (DH theta4) -->
+    <origin xyz="-$(arg a2) 0 0" rpy="0 0 0"/>
+    <axis xyz="0 1 0"/>
+    <limit lower="-6.28318530718" upper="6.28318530718" effort="$(arg joint_effort)" velocity="$(arg joint_vel)"/>
+    <dynamics damping="2.0" friction="0.0"/>
+  </joint>
+  <!-- joint4: wrist1 (about Y) at end of link3 (toward -X) -->
   <joint name="joint4" type="revolute">
     <parent link="link3"/>
-    <child link="frame4"/>
-    <origin xyz="0 0 0" rpy="0 0 0"/>
-    <axis xyz="0 0 1"/>
-    <limit lower="-6.28318530718" upper="6.28318530718" effort="$(arg joint_effort)" velocity="$(arg joint_vel)"/>
-    <dynamics damping="0.2" friction="0.0"/>
-  </joint>
-  <!-- DH after joint4: TransZ(d4) * RotX(+pi/2) -->
-  <joint name="dh4_fixed" type="fixed">
-    <parent link="frame4"/>
     <child link="link4"/>
-    <origin xyz="0 0 ${d4}" rpy="1.57079632679 0 0"/>
-  </joint>
-  <!-- Joint 5: rotation about Z (DH theta5) -->
+    <origin xyz="-$(arg a3) 0 0" rpy="0 0 0"/>
+    <axis xyz="0 1 0"/>
+    <limit lower="-6.28318530718" upper="6.28318530718" effort="$(arg joint_effort)" velocity="$(arg joint_vel)"/>
+    <dynamics damping="1.0" friction="0.0"/>
+  </joint>
+  <!-- joint5: wrist2 (about Z) at end of link4 (toward -Y) -->
   <joint name="joint5" type="revolute">
     <parent link="link4"/>
-    <child link="frame5"/>
-    <origin xyz="0 0 0" rpy="0 0 0"/>
+    <child link="link5"/>
+    <origin xyz="0 -$(arg d4) 0" rpy="0 0 0"/>
     <axis xyz="0 0 1"/>
     <limit lower="-6.28318530718" upper="6.28318530718" effort="$(arg joint_effort)" velocity="$(arg joint_vel)"/>
-    <dynamics damping="0.2" friction="0.0"/>
-  </joint>
-  <!-- DH after joint5: TransZ(d5) * RotX(-pi/2) -->
-  <joint name="dh5_fixed" type="fixed">
-    <parent link="frame5"/>
-    <child link="link5"/>
-    <origin xyz="0 0 ${d5}" rpy="-1.57079632679 0 0"/>
-  </joint>
-  <!-- Joint 6: rotation about Z (DH theta6) -->
+    <dynamics damping="1.0" friction="0.0"/>
+  </joint>
+  <!-- joint6: wrist3 (about Y) at end of link5 (along +Z) -->
   <joint name="joint6" type="revolute">
     <parent link="link5"/>
-    <child link="frame6"/>
-    <origin xyz="0 0 0" rpy="0 0 0"/>
-    <axis xyz="0 0 1"/>
-    <limit lower="-6.28318530718" upper="6.28318530718" effort="$(arg joint_effort)" velocity="$(arg joint_vel)"/>
-    <dynamics damping="0.2" friction="0.0"/>
-  </joint>
-  <!-- DH after joint6: TransZ(d6) -->
-  <joint name="dh6_fixed" type="fixed">
-    <parent link="frame6"/>
     <child link="link6"/>
-    <origin xyz="0 0 ${d6}" rpy="0 0 0"/>
-  </joint>
-  <!-- Tool -->
-  <joint name="tool0_fixed" type="fixed">
-    <parent link="link6"/>
-    <child link="tool0"/>
-    <origin xyz="0 0 0" rpy="0 0 0"/>
-  </joint>
-  <!--  ros2_control (gz_ros2_control) -->
+    <origin xyz="0 0 $(arg d5)" rpy="0 0 0"/>
+    <axis xyz="0 1 0"/>
+    <limit lower="-6.28318530718" upper="6.28318530718" effort="$(arg joint_effort)" velocity="$(arg joint_vel)"/>
+    <dynamics damping="0.8" friction="0.0"/>
+  </joint>
+  <!--
+       ros2_control (gz_ros2_control)
+        -->
   <ros2_control name="MyArmSystem" type="system">
     <hardware>

Commit message: ur5e7

File: src/my_arm_description/urdf/my_arm_ur5e2.urdf.xacro (robot description, xacro)
@@ -174,5 +174,5 @@
     <parent link="link3"/>
     <child link="link4"/>
-    <origin xyz="-$(arg a3) 0 0" rpy="0 0 0"/>
+    <origin xyz="-$(arg a3) 0 0" rpy="3.14159 0 0"/>
     <axis xyz="0 1 0"/>
     <limit lower="-6.28318530718" upper="6.28318530718" effort="$(arg joint_effort)" velocity="$(arg joint_vel)"/>

Commit message: ur5e7

File: src/my_arm_description/urdf/my_arm_ur5e2.urdf.xacro (robot description, xacro)
@@ -138,5 +138,5 @@
        link4 -> -Y, link5 -> -Z, link6 -> -Y -->
   <xacro:cyl_y name="link4" length="$(arg d4)" mass="$(arg m_link)" sign="-1"/>
-  <xacro:cyl_z name="link5" length="$(arg d5)" mass="$(arg m_link)"/>
+  <xacro:cyl_z name="link5" length="$(arg d5)" mass="$(arg m_link)" sign="-1"/>
   <xacro:cyl_y name="link6" length="$(arg d6)" mass="$(arg m_link)" sign="-1"/>
   <!--
@@ -174,5 +174,5 @@
     <parent link="link3"/>
     <child link="link4"/>
-    <origin xyz="-$(arg a3) 0 0" rpy="3.14159 0 0"/>
+    <origin xyz="-$(arg a3) 0 0" rpy="0 0 0"/>
     <axis xyz="0 1 0"/>
     <limit lower="-6.28318530718" upper="6.28318530718" effort="$(arg joint_effort)" velocity="$(arg joint_vel)"/>

Commit message: ur5e8

File: src/my_arm_description/urdf/my_arm_ur5e2.urdf.xacro (robot description, xacro)
@@ -88,12 +88,13 @@
         -->
   <xacro:macro name="cyl_z" params="name length mass">
+    <!-- sign: +1 or -1 to draw toward +Z or -Z -->
     <link name="${name}">
       <visual>
-        <origin xyz="0 0 ${length/2.0}" rpy="0 0 0"/>
+        <origin xyz="0 0 ${sign*length/2.0}" rpy="0 0 0"/>
         <geometry><cylinder radius="${r}" length="${length}"/></geometry>
         <material name="pale_blue"/>
       </visual>
       <collision>
-        <origin xyz="0 0 ${length/2.0}" rpy="0 0 0"/>
+        <origin xyz="0 0 ${sign*length/2.0}" rpy="0 0 0"/>
         <geometry><cylinder radius="${r}" length="${length}"/></geometry>
       </collision>

Commit message: ur5e9

File: src/my_arm_description/urdf/my_arm_ur5e2.urdf.xacro (robot description, xacro)
@@ -87,5 +87,5 @@
        Link macros (cylinders along x/y/z)
         -->
-  <xacro:macro name="cyl_z" params="name length mass">
+  <xacro:macro name="cyl_z" params="name length mass sign">
     <!-- sign: +1 or -1 to draw toward +Z or -Z -->
     <link name="${name}">
@@ -133,5 +133,5 @@
   </xacro:macro>
   <!-- Physical links -->
-  <xacro:cyl_z name="link1" length="$(arg d1)" mass="$(arg m_link)"/>
+  <xacro:cyl_z name="link1" length="$(arg d1)" mass="$(arg m_link)" sign="1"/>
   <xacro:cyl_x name="link2" length="$(arg a2)" mass="$(arg m_link)" sign="-1"/>
   <xacro:cyl_x name="link3" length="$(arg a3)" mass="$(arg m_link)" sign="-1"/>
@@ -193,5 +193,5 @@
     <parent link="link5"/>
     <child link="link6"/>
-    <origin xyz="0 0 $(arg d5)" rpy="0 0 0"/>
+    <origin xyz="0 0 -$(arg d5)" rpy="0 0 0"/>
     <axis xyz="0 1 0"/>
     <limit lower="-6.28318530718" upper="6.28318530718" effort="$(arg joint_effort)" velocity="$(arg joint_vel)"/>

Commit message: ur5e10

File: src/my_arm_description/urdf/my_arm_ur5e2.urdf.xacro (robot description, xacro)
@@ -63,4 +63,5 @@
   <material name="dark"><color rgba="0.2 0.2 0.2 1.0"/></material>
   <material name="pale_blue"><color rgba="0.6 0.75 0.95 1.0"/></material>
+  <material name="blue"><color rgba="0.2 0.3 0.8 1.0"/></material>
   <!--
        World + base
@@ -93,5 +94,5 @@
         <origin xyz="0 0 ${sign*length/2.0}" rpy="0 0 0"/>
         <geometry><cylinder radius="${r}" length="${length}"/></geometry>
-        <material name="pale_blue"/>
+        <material name="blue"/>
       </visual>
       <collision>
@@ -242,3 +243,12 @@
     </plugin>
   </gazebo>
+  <gazebo reference="link4">
+    <material>Gazebo/Blue</material>
+  </gazebo>
+    <gazebo reference="link5">
+    <material>Gazebo/Blue</material>
+  </gazebo>
+    <gazebo reference="link6">
+    <material>Gazebo/Blue</material>
+  </gazebo>
 </robot>
