Commit message: add puma and ur5e

File: src/my_arm_description/urdf/my_arm_puma.urdf.xacro (robot description, xacro)
@@ -138,6 +138,10 @@
   <xacro:wrist_link name="link6" mass="$(arg m_wrist)" mat="blue"/>
   <!-- =========================
-       Joints (6-DOF)
-       ========================= -->
+       Joints (6-DOF) - PUMA-like zero pose and rotation sense
+       Zero pose intent:
+         - Arm extended forward (+X), not vertical (+Z)
+         - q2,q3 positive => lift upward
+       ========================= -->
+  <!-- joint1: base yaw about +Z (standard) -->
   <joint name="joint1" type="revolute">
     <parent link="base_link"/>
@@ -148,21 +152,36 @@
     <dynamics damping="0.2" friction="0.0"/>
   </joint>
+  <!--
+    joint2: shoulder pitch
+    We rotate the joint frame so that link2 (a cylinder along its local +Z) points along +X at q2=0.
+    Rot_y(-90deg): local +Z becomes parent +X.
+    Also flip axis to make q2>0 lift (+X toward +Z).
+  -->
   <joint name="joint2" type="revolute">
     <parent link="link1"/>
     <child link="link2"/>
-    <origin xyz="0 0 ${L1}" rpy="0 0 0"/>
-    <axis xyz="0 1 0"/>
-    <limit lower="-3.14159" upper="3.14159" effort="$(arg joint_effort)" velocity="$(arg joint_vel)"/>
-    <dynamics damping="0.2" friction="0.0"/>
-  </joint>
+    <origin xyz="0 0 ${L1}" rpy="0 -1.57079632679 0"/>
+    <axis xyz="0 -1 0"/>
+    <limit lower="-3.14159" upper="3.14159" effort="$(arg joint_effort)" velocity="$(arg joint_vel)"/>
+    <dynamics damping="0.2" friction="0.0"/>
+  </joint>
+  <!--
+    joint3: elbow pitch
+    Keep the same sign convention as joint2: q3>0 lifts elbow upward.
+    No additional frame rotation needed: link2 frame already “forward”.
+  -->
   <joint name="joint3" type="revolute">
     <parent link="link2"/>
     <child link="link3"/>
     <origin xyz="0 0 ${L2}" rpy="0 0 0"/>
-    <axis xyz="0 1 0"/>
-    <limit lower="-3.14159" upper="3.14159" effort="$(arg joint_effort)" velocity="$(arg joint_vel)"/>
-    <dynamics damping="0.2" friction="0.0"/>
-  </joint>
-  <!-- Spherical wrist: all wrist joint origins coincide at the end of link3 -->
+    <axis xyz="0 -1 0"/>
+    <limit lower="-3.14159" upper="3.14159" effort="$(arg joint_effort)" velocity="$(arg joint_vel)"/>
+    <dynamics damping="0.2" friction="0.0"/>
+  </joint>
+  <!--
+    Spherical wrist at end of link3.
+    At q=0, forearm axis is link3 local +Z (which is “forward” in the world).
+    joint4: roll about forearm axis => use (0 0 1)
+  -->
   <joint name="joint4" type="revolute">
     <parent link="link3"/>
@@ -173,12 +192,14 @@
     <dynamics damping="0.2" friction="0.0"/>
   </joint>
+  <!-- joint5: wrist pitch (q5>0 “pitches up” with our sign choice) -->
   <joint name="joint5" type="revolute">
     <parent link="link4"/>
     <child link="link5"/>
     <origin xyz="0 0 0" rpy="0 0 0"/>
-    <axis xyz="0 1 0"/>
-    <limit lower="-3.14159" upper="3.14159" effort="$(arg joint_effort)" velocity="$(arg joint_vel)"/>
-    <dynamics damping="0.2" friction="0.0"/>
-  </joint>
+    <axis xyz="0 -1 0"/>
+    <limit lower="-3.14159" upper="3.14159" effort="$(arg joint_effort)" velocity="$(arg joint_vel)"/>
+    <dynamics damping="0.2" friction="0.0"/>
+  </joint>
+  <!-- joint6: wrist roll (tool roll) -->
   <joint name="joint6" type="revolute">
     <parent link="link5"/>

Commit message: xacro1

File: src/my_arm_description/urdf/my_arm_puma.urdf.xacro (robot description, xacro)
@@ -14,5 +14,5 @@
   <xacro:arg name="L6" default="0.0"/>
   <!-- Sizes -->
-  <xacro:arg name="r_link" default="0.02"/>
+  <xacro:arg name="r_link" default="0.01"/>
   <xacro:arg name="base_x" default="0.10"/>
   <xacro:arg name="base_y" default="0.10"/>
@@ -161,5 +161,5 @@
     <parent link="link1"/>
     <child link="link2"/>
-    <origin xyz="0 0 ${L1}" rpy="0 -1.57079632679 0"/>
+    <origin xyz="0 0 ${L1}" rpy="0 1.57079632679 0"/>
     <axis xyz="0 -1 0"/>
     <limit lower="-3.14159" upper="3.14159" effort="$(arg joint_effort)" velocity="$(arg joint_vel)"/>
@@ -174,5 +174,5 @@
     <parent link="link2"/>
     <child link="link3"/>
-    <origin xyz="0 0 ${L2}" rpy="0 0 0"/>
+    <origin xyz="0 0 ${L2}" rpy="0 57079632679 0"/>
     <axis xyz="0 -1 0"/>
     <limit lower="-3.14159" upper="3.14159" effort="$(arg joint_effort)" velocity="$(arg joint_vel)"/>

File: src/my_arm_description/urdf/my_arm_ur5e.urdf.xacro (robot description, xacro)
@@ -8,6 +8,6 @@
        ========================= -->
   <xacro:arg name="d1" default="0.1625"/>
-  <xacro:arg name="a2" default="-0.425"/>
-  <xacro:arg name="a3" default="-0.3922"/>
+  <xacro:arg name="a2" default="0.425"/>
+  <xacro:arg name="a3" default="0.3922"/>
   <xacro:arg name="d4" default="0.1333"/>
   <xacro:arg name="d5" default="0.0997"/>
@@ -33,6 +33,6 @@
   <xacro:property name="d5" value="$(arg d5)"/>
   <xacro:property name="d6" value="$(arg d6)"/>
-  <xacro:property name="a2_abs" value="${abs(a2)}"/>
-  <xacro:property name="a3_abs" value="${abs(a3)}"/>
+  <xacro:property name="a2_abs" value="$(arg a2)"/>
+  <xacro:property name="a3_abs" value="$(arg a3)"/>
   <xacro:property name="r"  value="$(arg r_link)"/>
   <!-- =========================

Commit message: xacro4

File: src/my_arm_description/urdf/my_arm_puma.urdf.xacro (robot description, xacro)
@@ -162,5 +162,5 @@
     <child link="link2"/>
     <origin xyz="0 0 ${L1}" rpy="0 1.57079632679 0"/>
-    <axis xyz="0 -1 0"/>
+    <axis xyz="0 1 0"/>
     <limit lower="-3.14159" upper="3.14159" effort="$(arg joint_effort)" velocity="$(arg joint_vel)"/>
     <dynamics damping="0.2" friction="0.0"/>
@@ -175,5 +175,5 @@
     <child link="link3"/>
     <origin xyz="0 0 ${L2}" rpy="0 57079632679 0"/>
-    <axis xyz="0 -1 0"/>
+    <axis xyz="0 1 0"/>
     <limit lower="-3.14159" upper="3.14159" effort="$(arg joint_effort)" velocity="$(arg joint_vel)"/>
     <dynamics damping="0.2" friction="0.0"/>

File: src/my_arm_description/urdf/my_arm_ur5e.urdf.xacro (robot description, xacro)
@@ -206,5 +206,5 @@
     <child link="link4"/>
     <origin xyz="${a3_abs} 0 0" rpy="-3.14 0 0"/>
-    <axis xyz="0 -1 0"/>
+    <axis xyz="0 1 0"/>
     <limit lower="-6.28318530718" upper="6.28318530718" effort="$(arg joint_effort)" velocity="$(arg joint_vel)"/>
     <dynamics damping="0.2" friction="0.0"/>
@@ -214,5 +214,5 @@
     <parent link="link4"/>
     <child link="link5"/>
-    <origin xyz="0 0 ${d4}" rpy="1.57 0 0"/>
+    <origin xyz="0 ${d4} 0" rpy="-1.57 0 0"/>
     <axis xyz="0 0 1"/>
     <limit lower="-6.28318530718" upper="6.28318530718" effort="$(arg joint_effort)" velocity="$(arg joint_vel)"/>
@@ -223,6 +223,6 @@
     <parent link="link5"/>
     <child link="link6"/>
-    <origin xyz="0 0 ${d5}" rpy="-1.57 0 0"/>
-    <axis xyz="0 -1 0"/>
+    <origin xyz="0 0 ${d5}" rpy="1.57 0 0"/>
+    <axis xyz="0 1 0"/>
     <limit lower="-6.28318530718" upper="6.28318530718" effort="$(arg joint_effort)" velocity="$(arg joint_vel)"/>
     <dynamics damping="0.2" friction="0.0"/>

Commit message: xacro puma ur5e

File: src/my_arm_description/urdf/my_arm_puma.urdf.xacro (robot description, xacro)
@@ -197,5 +197,5 @@
     <child link="link5"/>
     <origin xyz="0 0 0" rpy="0 0 0"/>
-    <axis xyz="0 -1 0"/>
+    <axis xyz="0 1 0"/>
     <limit lower="-3.14159" upper="3.14159" effort="$(arg joint_effort)" velocity="$(arg joint_vel)"/>
     <dynamics damping="0.2" friction="0.0"/>

File: src/my_arm_description/urdf/my_arm_ur5e.urdf.xacro (robot description, xacro)
@@ -154,5 +154,5 @@
   <link name="tool0">
     <visual>
-      <origin xyz="0 0 0.02" rpy="0 0 0"/>
+      <origin xyz="0 0 0" rpy="0 0 0"/>
       <geometry>
         <box size="0.05 0.05 0.04"/>

Commit message: xacro3

File: src/my_arm_description/urdf/my_arm_puma.urdf.xacro (robot description, xacro)
@@ -6,7 +6,7 @@
        ========================= -->
   <!-- Link lengths (meters) -->
-  <xacro:arg name="L1" default="0.12"/>
-  <xacro:arg name="L2" default="0.12"/>
-  <xacro:arg name="L3" default="0.12"/>
+  <xacro:arg name="L1" default="0.4"/>
+  <xacro:arg name="L2" default="0.4318"/>
+  <xacro:arg name="L3" default="0.43208"/>
   <!-- Spherical wrist: set these to 0 -->
   <xacro:arg name="L4" default="0.0"/>
@@ -17,5 +17,5 @@
   <xacro:arg name="base_x" default="0.10"/>
   <xacro:arg name="base_y" default="0.10"/>
-  <xacro:arg name="base_z" default="0.04"/>
+  <xacro:arg name="base_z" default="0.02"/>
   <!-- Masses (kg) -->
   <xacro:arg name="m_base" default="1.0"/>
@@ -26,4 +26,5 @@
   <xacro:arg name="joint_effort" default="5.0"/>
   <!-- Convenience properties -->
+  <xacro:property name="base_z" value="$(arg base_z)"/>
   <xacro:property name="L1" value="$(arg L1)"/>
   <xacro:property name="L2" value="$(arg L2)"/>
@@ -75,5 +76,5 @@
     <parent link="world"/>
     <child link="base_link"/>
-    <origin xyz="0 0 0" rpy="0 0 0"/>
+    <origin xyz="0 0 ${base_z}" rpy="0 0 0"/>
   </joint>
   <link name="base_link">
@@ -147,5 +148,5 @@
     <parent link="base_link"/>
     <child link="link1"/>
-    <origin xyz="0 0 $(arg base_z)" rpy="0 0 0"/>
+    <origin xyz="0 0 ${L1}" rpy="0 0 0"/>
     <axis xyz="0 0 1"/>
     <limit lower="-3.14159" upper="3.14159" effort="$(arg joint_effort)" velocity="$(arg joint_vel)"/>
@@ -161,5 +162,5 @@
     <parent link="link1"/>
     <child link="link2"/>
-    <origin xyz="0 0 ${L1}" rpy="0 1.57079632679 0"/>
+    <origin xyz="0 0 0" rpy="0 1.57079632679 0"/>
     <axis xyz="0 1 0"/>
     <limit lower="-3.14159" upper="3.14159" effort="$(arg joint_effort)" velocity="$(arg joint_vel)"/>
@@ -174,5 +175,5 @@
     <parent link="link2"/>
     <child link="link3"/>
-    <origin xyz="0 0 ${L2}" rpy="0 57079632679 0"/>
+    <origin xyz="0 0 ${L2}" rpy="0 1.57079632679 0"/>
     <axis xyz="0 1 0"/>
     <limit lower="-3.14159" upper="3.14159" effort="$(arg joint_effort)" velocity="$(arg joint_vel)"/>

Commit message: puma no DH

File: src/my_arm_description/urdf/my_arm_puma.urdf.xacro (robot description, xacro)
@@ -26,5 +26,4 @@
   <xacro:arg name="joint_effort" default="5.0"/>
   <!-- Convenience properties -->
-  <xacro:property name="base_z" value="$(arg base_z)"/>
   <xacro:property name="L1" value="$(arg L1)"/>
   <xacro:property name="L2" value="$(arg L2)"/>
@@ -76,5 +75,5 @@
     <parent link="world"/>
     <child link="base_link"/>
-    <origin xyz="0 0 ${base_z}" rpy="0 0 0"/>
+    <origin xyz="0 0 $(arg base_z)" rpy="0 0 0"/>
   </joint>
   <link name="base_link">
@@ -148,5 +147,5 @@
     <parent link="base_link"/>
     <child link="link1"/>
-    <origin xyz="0 0 ${L1}" rpy="0 0 0"/>
+    <origin xyz="0 0 0" rpy="0 0 0"/>
     <axis xyz="0 0 1"/>
     <limit lower="-3.14159" upper="3.14159" effort="$(arg joint_effort)" velocity="$(arg joint_vel)"/>
@@ -162,5 +161,5 @@
     <parent link="link1"/>
     <child link="link2"/>
-    <origin xyz="0 0 0" rpy="0 1.57079632679 0"/>
+    <origin xyz="0 0 ${L1}" rpy="0 1.57079632679 0"/>
     <axis xyz="0 1 0"/>
     <limit lower="-3.14159" upper="3.14159" effort="$(arg joint_effort)" velocity="$(arg joint_vel)"/>
@@ -175,5 +174,5 @@
     <parent link="link2"/>
     <child link="link3"/>
-    <origin xyz="0 0 ${L2}" rpy="0 1.57079632679 0"/>
+    <origin xyz="0 0 ${L2}" rpy="0 -1.57079632679 0"/>
     <axis xyz="0 1 0"/>
     <limit lower="-3.14159" upper="3.14159" effort="$(arg joint_effort)" velocity="$(arg joint_vel)"/>

Commit message: puma2

File: src/my_arm_description/urdf/my_arm_puma.urdf.xacro (robot description, xacro)
@@ -9,4 +9,5 @@
   <xacro:arg name="L2" default="0.4318"/>
   <xacro:arg name="L3" default="0.43208"/>
+  <xacro:arg name="d3" default="0.1397"/>
   <!-- Spherical wrist: set these to 0 -->
   <xacro:arg name="L4" default="0.0"/>
@@ -14,5 +15,5 @@
   <xacro:arg name="L6" default="0.0"/>
   <!-- Sizes -->
-  <xacro:arg name="r_link" default="0.01"/>
+  <xacro:arg name="r_link" default="0.03"/>
   <xacro:arg name="base_x" default="0.10"/>
   <xacro:arg name="base_y" default="0.10"/>
@@ -30,4 +31,5 @@
   <xacro:property name="L3" value="$(arg L3)"/>
   <xacro:property name="r"  value="$(arg r_link)"/>
+  <xacro:property name="d3" value="$(arg d3)"/>
   <!-- Wrist visualization radius (small spheres) -->
   <xacro:property name="r_wrist" value="${0.5 * $(arg r_link)}"/>
@@ -67,4 +69,5 @@
   <material name="dark"><color rgba="0.2 0.2 0.2 1.0"/></material>
   <material name="blue"><color rgba="0.2 0.3 0.8 1.0"/></material>
+  <material name="pale_blue"><color rgba="0.70 0.82 1.00 1.0"/></material>
   <!-- =========================
        Links
@@ -112,7 +115,7 @@
     </link>
   </xacro:macro>
-  <xacro:arm_link name="link1" length="${L1}" mass="$(arg m_link)" mat="grey"/>
-  <xacro:arm_link name="link2" length="${L2}" mass="$(arg m_link)" mat="grey"/>
-  <xacro:arm_link name="link3" length="${L3}" mass="$(arg m_link)" mat="grey"/>
+  <xacro:arm_link name="link1" length="${L1}" mass="$(arg m_link)" mat="pale_blue"/>
+  <xacro:arm_link name="link2" length="${L2}" mass="$(arg m_link)" mat="pale_blue"/>
+  <xacro:arm_link name="link3" length="${L3}" mass="$(arg m_link)" mat="pale_blue"/>
   <!-- Wrist links: zero-length, just small spheres to visualize axes -->
   <xacro:macro name="wrist_link" params="name mass mat">
@@ -161,5 +164,5 @@
     <parent link="link1"/>
     <child link="link2"/>
-    <origin xyz="0 0 ${L1}" rpy="0 1.57079632679 0"/>
+    <origin xyz="0 ${d3} ${L1}" rpy="0 1.57079632679 0"/>
     <axis xyz="0 1 0"/>
     <limit lower="-3.14159" upper="3.14159" effort="$(arg joint_effort)" velocity="$(arg joint_vel)"/>
@@ -256,3 +259,12 @@
     </plugin>
   </gazebo>
+  <gazebo reference="link1">
+    <material>Gazebo/LightBlue</material>
+  </gazebo>
+  <gazebo reference="link2">
+    <material>Gazebo/LightBlue</material>
+  </gazebo>
+  <gazebo reference="link3">
+    <material>Gazebo/LightBlue</material>
+  </gazebo>
 </robot>

Commit message: gz_sim1

File: src/my_arm_description/urdf/my_arm_puma.urdf.xacro (robot description, xacro)
@@ -15,5 +15,5 @@
   <xacro:arg name="L6" default="0.0"/>
   <!-- Sizes -->
-  <xacro:arg name="r_link" default="0.03"/>
+  <xacro:arg name="r_link" default="0.04"/>
   <xacro:arg name="base_x" default="0.10"/>
   <xacro:arg name="base_y" default="0.10"/>
@@ -260,11 +260,11 @@
   </gazebo>
   <gazebo reference="link1">
-    <material>Gazebo/LightBlue</material>
+    <material>Gazebo/Blue</material>
   </gazebo>
   <gazebo reference="link2">
-    <material>Gazebo/LightBlue</material>
+    <material>Gazebo/Blue</material>
   </gazebo>
   <gazebo reference="link3">
-    <material>Gazebo/LightBlue</material>
+    <material>Gazebo/Blue</material>
   </gazebo>
 </robot>

Commit message: urdf puma2

File: src/my_arm_description/urdf/my_arm_puma.urdf.xacro (robot description, xacro)
@@ -122,13 +122,13 @@
     <xacro:inertial_cylinder_x mass="$(arg m_link)" radius="${r}" length="${L2}"/>
   </link>
-  <!-- link3: visually along +X -->
+  <!-- link3: visually along +Z -->
   <link name="link3">
     <visual>
-      <origin xyz="${L3/2.0} 0 0" rpy="0 1.57079632679 0"/>
+      <origin xyz="${L3/2.0} 0 0" rpy="0 0 0"/>
       <geometry><cylinder radius="${r}" length="${L3}"/></geometry>
       <material name="pale_blue"/>
     </visual>
     <collision>
-      <origin xyz="${L3/2.0} 0 0" rpy="0 1.57079632679 0"/>
+      <origin xyz="${L3/2.0} 0 0" rpy="0 0 0"/>
       <geometry><cylinder radius="${r}" length="${L3}"/></geometry>
     </collision>

Commit message: urdf puma3

File: src/my_arm_description/urdf/my_arm_puma.urdf.xacro (robot description, xacro)
@@ -101,5 +101,5 @@
       <origin xyz="0 0 ${L1/2.0}" rpy="0 0 0"/>
       <geometry><cylinder radius="${r}" length="${L1}"/></geometry>
-      <material name="pale_blue"/>
+      <material name="blue"/>
     </visual>
     <collision>
@@ -125,10 +125,10 @@
   <link name="link3">
     <visual>
-      <origin xyz="${L3/2.0} 0 0" rpy="0 0 0"/>
+      <origin xyz="0 0 ${L3/2.0}" rpy="0 0 0"/>
       <geometry><cylinder radius="${r}" length="${L3}"/></geometry>
       <material name="pale_blue"/>
     </visual>
     <collision>
-      <origin xyz="${L3/2.0} 0 0" rpy="0 0 0"/>
+      <origin xyz="0 0 ${L3/2.0}" rpy="0 0 0"/>
       <geometry><cylinder radius="${r}" length="${L3}"/></geometry>
     </collision>
@@ -189,5 +189,5 @@
     <parent link="link3"/>
     <child link="link4"/>
-    <origin xyz="${L3} 0 0" rpy="0 0 0"/>
+    <origin xyz="0 0 ${L3}" rpy="0 0 0"/>
     <axis xyz="0 0 1"/>
     <limit lower="-3.14159" upper="3.14159" effort="$(arg joint_effort)" velocity="$(arg joint_vel)"/>
